File: Final Project/ECE414_Final_Proj/ECE414_Final_Proj/ECE414_Final_Proj.kicad_sch (KiCad schematic)
At the start: 0 parts

Commit message: project progress
Other:
- company: (none) -> ECE 414
- title: (none) -> Sam_Sam_David_Synthesizer
Changed lines of the file:
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@@
 	(generator_version "8.0")
 	(paper "A4")
+	(title_block
+		(title "Sam_Sam_David_Synthesizer")
+		(company "ECE 414")
+	)
 	(sheet
 		(at 86.36 24.13)
