File: Final Project/ECE414_Final_Proj/ECE414_Final_Proj/Analog Inputs.kicad_sch (KiCad schematic)
At the start: 34 parts, among them U17 MCP3008, U18 MCP3008

Commit message: we made the schematic happy
Parts:
- R15: value FSR -> C-FSR
- R17: value FSR -> D_FSR
- R19: value FSR -> E_FSR
- R23: value FSR -> F_FSR
- R25: value FSR -> G_FSR
- R27: value FSR -> A_FSR
- R29: value FSR -> B_FSR
- R31: value FSR -> C#_FSR
- R33: value FSR -> D#_FSR
- R35: value FSR -> F#_FSR
- R37: value FSR -> G#_FSR
- R39: value FSR -> A#_FSR
- R41: value FSR -> Decay Adjust
- R43: value FSR -> Attack Adjust
- R45: value FSR -> Extra Slider Fun
- R47: value FSR -> Volume Slider
- renumbered U17 to ADC_1, U18 to ADC_2
Connections:
- net CS_ADC_2: now reaches ADC_2.10 (~{CS}/SHDN)
- net SDO_SPI1: now reaches ADC_2.11 (Din)
- net SDO_SPI1: now also ADC_1.11 (Din)
- net SDI_SPI1: now reaches ADC_2.12 (Dout)
- net SDI_SPI1: now also ADC_1.12 (Dout)
- net CLK_SPI1: now reaches ADC_2.13 (CLK)
- net CLK_SPI1: now also ADC_1.13 (CLK)
- net CS_ADC_1: now reaches ADC_1.10 (~{CS}/SHDN)
Other:
- moved on the sheet: ADC_1, ADC_2, R15, R16, R17, R18, R19, R22, R23, R24, R25, R26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

Commit message: project progress
Connections:
- net 3V3: now also ADC_1.15 (Vref), ADC_1.16 (Vdd), ADC_2.15 (Vref), ADC_2.16 (Vdd)
Other:
- company: (none) -> ECE 414
- title: (none) -> Sam_Sam_David_Synthesizer
- moved on the sheet: ADC_1, ADC_2, R15, R16, R17, R18, R19, R22, R23, R24, R25, R26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

Commit message: Other fixin's
Parts:
- removed R43: Attack Adjust, symbol Device:R_Variable_US
- removed R44, R46, R48: 10K, symbol Device:R_US
- removed R45: Extra Slider Fun, symbol Device:R_Variable_US
- removed R47: Volume Slider, symbol Device:R_Variable_US
