File: Final Project/ECE414_Final_Proj/ECE414_Final_Proj/untitled.kicad_sch (KiCad schematic)
At the start: 27 parts, among them J2 AudioJack2_SwitchT, SW2 SW_Push, U1 TXS0108EPW, U10 RPi Pico, U11 74HC595, U12 YM3812, U13 YM3014B, U15 TL072, U3B1 TL072, U9 LT1086-ADJ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

Commit message: Schematic Work Update
Parts:
- removed C12: 0.1uF, symbol Device:C_Small
- added C1, C2: 0.1uF, symbol Device:C_Small
Connections:
- net GNDREF: now also C1.1, C2.1
- net VDD: now also C16.2, U13.1 (VDD), C1.2, C2.2
- net at C17.1, U3B1.1: now also U3B1.2 (-); no longer U3B1.3 (+)
- net at U12.20 (S&H): now also U13.3 (LOAD)
- net at U12.21 (M0): now also U13.4 (SD)
- net at U12.23 (SY): now also U13.5 (CLOCK)
- net at U12.3 (~{IC}): now also U1.16 (B4)
- net at U12.4 (A0): now also U1.15 (B5)
- net at U12.5 (~{WR}): now also U1.14 (B6)
- net at U12.7 (~{CS}): now also U1.13 (B7)
- net at U11.12 (RCLK): now also U1.17 (B3)
- net at U10.10 (GP7): now also U1.4 (A3)
- net at U10.25 (GP19): now also U1.8 (A7)
- net at U10.26 (GP20): now also U1.7 (A6)
- net at U10.27 (GP21): now also U1.6 (A5)
- net at U10.29 (GP22): now also U1.5 (A4)
- net at C18.1, U13.7 (RB): now also U15.3 (+); no longer U15.2 (-)
- net at U13.2 (BUFF): now also U3B1.3 (+)
- net at C19.1, U13.8 (MP), U15.1: now also U15.2 (-); no longer U15.3 (+)
- no-connect marks 1 -> 3
Other:
- moved on the sheet: U15A

Commit message: we made the schematic happy
Connections:
- net CS_ADC_2: now reaches U10.12 (GP9)
- net SPI_1_CLK: now reaches U10.14 (GP10)
- net SDO_SPI1: now reaches U10.15 (GP11)
- net SDI_SP1: now reaches U10.16 (GP12)
- net CS_ADC_1: now reaches U10.17 (GP13)
Changed lines of the file:
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@@
+	(wire
+		(pts
+			(xy 45.72 168.91) (xy 53.34 168.91)
+		)
+		(stroke
+			(width 0)
+			(type default)
+		)
+	)
 	(wire
 		(pts
@@
 	(wire
 		(pts
+			(xy 104.14 138.43) (xy 107.95 138.43)
+		)
+		(stroke
+			(width 0)
+			(type default)
+		)
+	)
+	(wire
+		(pts
 			(xy 232.41 156.21) (xy 232.41 215.9)
 		)
@@
 		)
 	)
+	(wire
+		(pts
+			(xy 44.45 163.83) (xy 53.34 163.83)
+		)
+		(stroke
+			(width 0)
+			(type default)
+		)
+	)
 	(bus
 		(pts
@@
 	(wire
 		(pts
+			(xy 45.72 161.29) (xy 53.34 161.29)
+		)
+		(stroke
+			(width 0)
+			(type default)
+		)
+	)
+	(wire
+		(pts
 			(xy 241.3 148.59) (xy 220.98 148.59)
 		)
@@
 		(pts
 			(xy 261.62 153.67) (xy 265.43 153.67)
+		)
+		(stroke
+			(width 0)
+			(type default)
+		)
+	)
+	(wire
+		(pts
+			(xy 45.72 166.37) (xy 53.34 166.37)
 		)
 		(stroke
@@
 		)
 	)
+	(global_label "SDI_SP1"
+		(shape input)
+		(at 45.72 168.91 180)
+		(fields_autoplaced yes)
+		(effects
+			(font
+				(size 1.27 1.27)
+			)
+			(justify right)
+		)
+		(property "Intersheetrefs" "${INTERSHEET_REFS}"
+			(at 34.9939 168.91 0)
+			(effects
+				(font
+					(size 1.27 1.27)
+				)
+				(justify right)
+				(hide yes)
+			)
+		)
+	)
 	(global_label "3V3"
 		(shape input)
@@
 		)
 	)
+	(global_label "SPI_1_CLK"
+		(shape input)
+		(at 44.45 163.83 180)
+		(fields_autoplaced yes)
+		(effects
+			(font
+				(size 1.27 1.27)
+			)
+			(justify right)
+		)
+		(property "Intersheetrefs" "${INTERSHEET_REFS}"
+			(at 31.6677 163.83 0)
+			(effects
+				(font
+					(size 1.27 1.27)
+				)
+				(justify right)
+				(hide yes)
+			)
+		)
+	)
+	(global_label "CS_ADC_1"
+		(shape input)
+		(at 107.95 138.43 0)
+		(fields_autoplaced yes)
+		(effects
+			(font
+				(size 1.27 1.27)
+			)
+			(justify left)
+		)
+		(property "Intersheetrefs" "${INTERSHEET_REFS}"
+			(at 120.188 138.43 0)
+			(effects
+				(font
+					(size 1.27 1.27)
+				)
+				(justify left)
+				(hide yes)
+			)
+		)
+	)
 	(global_label "3V3"
 		(shape input)
@@
 				(hide yes)
 			)
+		)
+	)
+	(global_label "CS_ADC_2"
+		(shape input)
+		(at 45.72 161.29 180)
+		(fields_autoplaced yes)
+		(effects
+			(font
+				(size 1.27 1.27)
+			)
+			(justify right)
+		)
+		(property "Intersheetrefs" "${INTERSHEET_REFS}"
+			(at 33.482 161.29 0)
+			(effects
+				(font
+					(size 1.27 1.27)
+				)
+				(justify right)
+				(hide yes)
+			)
+		)
+	)
+	(global_label "SDO_SPI1"
+		(shape input)
+		(at 45.72 166.37 180)
+		(fields_autoplaced yes)
+		(effects
+			(font
+				(size 1.27 1.27)
+			)
+			(justify right)
+		)
+		(property "Intersheetrefs" "${INTERSHEET_REFS}"
+			(at 33.6634 166.37 0)
+			(effects
+				(font
+					(size 1.27 1.27)
+				)
+				(justify right)
+				(hide yes)
+			)

Commit message: we made the schematic sad again
Parts:
- added D1: Power Indicator LED, symbol Device:LED
- added D2, D3, D4, D5: LED, symbol Device:LED
- added R2: 220, symbol Device:R_US
- added R3, R4, R5, R6: R_US, symbol Device:R_US
- added SW1: SW_Push_Left, symbol Switch:SW_Push
- added SW3: SW_Push_Enter, symbol Switch:SW_Push
- added SW4: SW_Push_Right, symbol Switch:SW_Push
- added U2: 74HC595, symbol 74xx:74HC595
Connections:
- net GNDREF: now also D1.1 (K), D2.1 (K), D3.1 (K), D4.1 (K), D5.1 (K), SW1.2, SW3.2, SW4.2
- net VDD: now also R2.1
- new net: D1.2 (A), R2.2
- new net: R5.1, U2.3 (QD)
- new net: D4.2 (A), R5.2
- new net: R4.1, U2.2 (QC)
- new net: D3.2 (A), R4.2
- new net: SW3.1, U2.6 (QG)
- new net: R3.1, U2.1 (QB)
- new net: R6.1, U2.4 (QE)
- new net: SW1.1, U2.5 (QF)
- new net: SW4.1, U2.7 (QH)
- new net: D2.2 (A), R3.2
- new net: D5.2 (A), R6.2

Commit message: project progress
Parts:
- removed D2, D3, D4, D5: LED, symbol Device:LED
- removed R3, R4, R5, R6: R_US, symbol Device:R_US
- removed SW1: SW_Push_Left, symbol Switch:SW_Push
- removed SW3: SW_Push_Enter, symbol Switch:SW_Push
- removed U2: 74HC595, symbol 74xx:74HC595
- added D6: LED_BKGR, symbol Device:LED_BKGR
- added R7, R8, R9: R_US, symbol Device:R_US
- SW4: value SW_Push_Right -> SW_Push_Clockwise
Connections:
- net GNDREF: now also D6.2 (K)
- net at SW4.1: now also U10.9 (GP6)
- net at U10.31 (GP26): now also R7.2
- net at U10.32 (GP27): now also R8.2
- net at U10.34 (GP28): now also R9.2
- new net: D6.3 (GA), R8.1
- new net: D6.1 (BA), R9.1
- new net: D6.4 (RA), R7.1
Other:
- company: (none) -> ECE 414
- title: (none) -> Sam_Sam_David_Synthesizer
- moved on the sheet: C1, C11, C13, C14, C15, C16, C17, C18, C19, C2, C2-Tant1, C20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

Commit message: Updated Schematic and General Cleanup
Parts:
- added C3: 0.1uF, symbol Device:C_Small
- added R3: 1M, symbol Device:R_US
- added R4: 220, symbol Device:R_US
- added U2: 74HC04, symbol 74xx:74HC04
Connections:
- net GNDREF: now also C14.2, U10.A (USB_SHIELD), U10.B (USB_SHIELD), U10.C (USB_SHIELD), U10.D (USB_SHIELD), C3.1, U2.7 (GND); no longer C14.1
- net VDD: now also C3.2, U2.14 (VCC)
- net at C15.2, Y2.2: now also R3.1, U2.1
- net 12V Unregulated renamed 6.5V Unregulated
- new net: C14.1, R3.2, R4.1, Y2.1
- new net: R4.2, U2.2, U2.3
- new net 3.58 MHz: U12.24 (MCLK), U2.4
Other:
- moved on the sheet: C14, C15, Y2

Commit message: Other fixin's
Parts:
- removed D6: LED_BKGR, symbol Device:LED_BKGR
- removed R7, R8, R9: R_US, symbol Device:R_US
- added SW1: Vibrato, symbol Switch:SW_Push
Connections:
- net GNDREF: now also SW1.2
- net at U10.34 (GP28): now also SW1.1
